File: nautilus-board.sch (EAGLE design)
At the start: 35 parts, among them Q3 DMG2305, SW1 KMR2, U1 2MB Flash, U2 AP2112(3.3V), U3 MCP73831T-2ACI/OT, X1 JSTPH, X2 4u20329

Commit message: External XTAL
Parts:
- added C2, C3: 22pF, microbuilder:CAP_CERAMIC0603_NO
- added Y2: 32.768, adafruit2:XTAL-3.2X1.5
Connections:
- removed net A5: MS1.GPIO13, U$1.P0.05/AIN3
- new net N$2: C3.1, U$1.P0.01/XTAL2, Y2.P$2
- new net N$7: C2.1, U$1.P0.00/XTAL1, Y2.P$1
- net D2: no longer MS1.GPIOA4
- net D3: no longer U$1.P1.09
- net GND: now also C2.2, C3.2
- net NEOPIXEL: now also U$1.P1.09; no longer U$1.P0.00/XTAL1
- net VDIV: now also U$1.P0.05/AIN3; no longer U$1.P0.01/XTAL2
Other:
- note added: "D3, A5"
- note removed: "We'll use the internal crystal connected to XC2, XC1"
- note removed: "XTAL"
Changed lines of the file:
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@@
 <drawing>
 <settings>
-<setting alwaysvectorfont="yes"/>
+<setting alwaysvectorfont="no"/>
 <setting verticaltext="up"/>
 </settings>
@@
 <part name="C10" library="microbuilder" deviceset="CAP_CERAMIC" device="0603_NO" value="0.1uF"/>
 <part name="U$5" library="microbuilder" deviceset="GND" device=""/>
+<part name="U$17" library="microbuilder" deviceset="GND" device=""/>
+<part name="Y2" library="adafruit2" deviceset="XTAL" device="-3.2X1.5" value="32.768"/>
+<part name="C2" library="microbuilder" deviceset="CAP_CERAMIC" device="0603_NO" value="22pF"/>
+<part name="C3" library="microbuilder" deviceset="CAP_CERAMIC" device="0603_NO" value="22pF"/>
 </parts>
 <sheets>
@@
 <text x="195.58" y="17.78" size="1.778" layer="94">RED LED</text>
 <text x="215.9" y="17.78" size="1.778" layer="94">RESET</text>
-<text x="63.5" y="96.52" size="1.778" layer="94">XTAL</text>
-<text x="71.12" y="91.44" size="1.27" layer="97" align="center">We'll use the internal
-crystal connected to XC2, XC1</text>
 <text x="109.22" y="91.44" size="1.778" layer="94">MICRO USB</text>
 <text x="187.96" y="-40.64" size="1.778" layer="94">SPI Flash</text>
@@
 300mA: ~300/~125mV
 600mA: ~375/~260mV</text>
+<text x="2.54" y="88.9" size="1.778" layer="91">D3, A5</text>
 </plain>
 <instances>
@@
 <instance part="U$5" gate="G$1" x="63.5" y="142.24" smashed="yes">
 <attribute name="VALUE" x="61.976" y="139.7" size="1.27" layer="96"/>
+</instance>
+<instance part="U$17" gate="G$1" x="91.44" y="119.38" smashed="yes" rot="R180">
+<attribute name="VALUE" x="92.964" y="121.92" size="1.27" layer="96" rot="R180"/>
+</instance>
+<instance part="Y2" gate="G$1" x="73.66" y="116.84" smashed="yes" rot="R90">
+<attribute name="NAME" x="69.85" y="114.3" size="1.27" layer="95" font="vector" rot="R90"/>
+<attribute name="VALUE" x="78.74" y="113.03" size="1.27" layer="96" font="vector" rot="R90"/>
+</instance>
+<instance part="C2" gate="G$1" x="83.82" y="109.22" smashed="yes" rot="R90">
+<attribute name="NAME" x="82.57" y="106.93" size="1.27" layer="95" font="vector" rot="R180" align="center"/>
+<attribute name="VALUE" x="82.57" y="111.52" size="1.27" layer="96" font="vector" rot="R180" align="center"/>
+</instance>
+<instance part="C3" gate="G$1" x="83.82" y="124.46" smashed="yes" rot="R90">
+<attribute name="NAME" x="82.57" y="122.17" size="1.27" layer="95" font="vector" rot="R180" align="center"/>
+<attribute name="VALUE" x="82.57" y="126.76" size="1.27" layer="96" font="vector" rot="R180" align="center"/>
 </instance>
 </instances>
@@
 <pinref part="U$5" gate="G$1" pin="GND"/>
 <wire x1="63.5" y1="144.78" x2="63.5" y2="147.32" width="0.1524" layer="91"/>
+</segment>
+<segment>
+<pinref part="U$17" gate="G$1" pin="GND"/>
+<wire x1="91.44" y1="116.84" x2="91.44" y2="114.3" width="0.1524" layer="91"/>
+<wire x1="86.36" y1="109.22" x2="88.9" y2="109.22" width="0.1524" layer="91"/>
+<wire x1="88.9" y1="109.22" x2="88.9" y2="114.3" width="0.1524" layer="91"/>
+<wire x1="88.9" y1="114.3" x2="88.9" y2="124.46" width="0.1524" layer="91"/>
+<wire x1="88.9" y1="124.46" x2="86.36" y2="124.46" width="0.1524" layer="91"/>
+<wire x1="91.44" y1="114.3" x2="88.9" y2="114.3" width="0.1524" layer="91"/>
+<junction x="88.9" y="114.3"/>
+<pinref part="C2" gate="G$1" pin="2"/>
+<pinref part="C3" gate="G$1" pin="2"/>
 </segment>
 </net>
@@
 </segment>
 <segment>
-<pinref part="U$1" gate="G$1" pin="P0.00/XTAL1"/>
-<wire x1="53.34" y1="73.66" x2="53.34" y2="114.3" width="0.1524" layer="91"/>
-<label x="53.34" y="99.06" size="1.778" layer="95" rot="R90"/>
+<pinref part="U$1" gate="G$1" pin="P1.09"/>
+<wire x1="38.1" y1="73.66" x2="38.1" y2="93.98" width="0.1524" layer="91"/>
+<label x="38.1" y="101.6" size="1.778" layer="95"/>
 </segment>
 </net>
@@
 <net name="VDIV" class="0">
 <segment>
-<pinref part="U$1" gate="G$1" pin="P0.01/XTAL2"/>
-<wire x1="48.26" y1="73.66" x2="48.26" y2="111.76" width="0.1524" layer="91"/>
-<label x="48.26" y="88.9" size="1.778" layer="95" rot="R90"/>
-</segment>
-<segment>
 <wire x1="-68.58" y1="137.16" x2="-68.58" y2="134.62" width="0.1524" layer="91"/>
 <wire x1="-68.58" y1="134.62" x2="-68.58" y2="132.08" width="0.1524" layer="91"/>
@@
 <pinref part="R12" gate="G$3" pin="2"/>
 </segment>
+<segment>
+<pinref part="U$1" gate="G$1" pin="P0.05/AIN3"/>
+<wire x1="43.18" y1="73.66" x2="43.18" y2="93.98" width="0.1524" layer="91"/>
+<label x="43.18" y="93.98" size="1.778" layer="95"/>
+</segment>
 </net>
 <net name="A0" class="0">
@@
 </segment>
 </net>
-<net name="A5" class="0">
-<segment>
-<pinref part="U$1" gate="G$1" pin="P0.05/AIN3"/>
-<wire x1="43.18" y1="73.66" x2="43.18" y2="111.76" width="0.1524" layer="91"/>
-<label x="43.18" y="88.9" size="1.778" layer="95" rot="R90"/>
-</segment>
-<segment>
-<pinref part="MS1" gate="G$1" pin="GPIO13"/>
-<wire x1="-81.28" y1="-15.24" x2="-66.04" y2="-15.24" width="0.1524" layer="91"/>
-<label x="-76.2" y="-15.24" size="1.778" layer="95"/>
-</segment>
-</net>
 <net name="D1" class="0">
 <segment>
@@
 <net name="D2" class="0">
 <segment>
-<pinref part="MS1" gate="G$1" pin="GPIOA4"/>
-<wire x1="-124.46" y1="-17.78" x2="-132.08" y2="-17.78" width="0.1524" layer="91"/>
-<label x="-129.54" y="-17.78" size="1.778" layer="95"/>
-</segment>
-<segment>
 <pinref part="U$1" gate="G$1" pin="P0.07"/>
 <wire x1="-5.08" y1="-43.18" x2="-20.32" y2="-43.18" width="0.1524" layer="91"/>
@@
 </net>
 <net name="D3" class="0">
-<segment>
-<pinref part="U$1" gate="G$1" pin="P1.09"/>
-<wire x1="38.1" y1="73.66" x2="38.1" y2="111.76" width="0.1524" layer="91"/>
-<label x="38.1" y="88.9" size="1.778" layer="95" rot="R90"/>
-</segment>
 <segment>
 <pinref part="MS1" gate="G$1" pin="GPIOA3"/>
@@
 </segment>
 </net>
+<net name="N$7" class="0">
+<segment>
+<wire x1="78.74" y1="109.22" x2="73.66" y2="109.22" width="0.1524" layer="91"/>
+<pinref part="Y2" gate="G$1" pin="P$1"/>
+<wire x1="73.66" y1="109.22" x2="73.66" y2="111.76" width="0.1524" layer="91"/>
+<junction x="73.66" y="109.22"/>
+<pinref part="C2" gate="G$1" pin="1"/>
+<pinref part="U$1" gate="G$1" pin="P0.00/XTAL1"/>
+<wire x1="53.34" y1="73.66" x2="53.34" y2="109.22" width="0.1524" layer="91"/>
+<wire x1="53.34" y1="109.22" x2="73.66" y2="109.22" width="0.1524" layer="91"/>
+</segment>
+</net>
+<net name="N$2" class="0">
+<segment>
+<pinref part="Y2" gate="G$1" pin="P$2"/>
+<wire x1="78.74" y1="124.46" x2="73.66" y2="124.46" width="0.1524" layer="91"/>
+<wire x1="73.66" y1="124.46" x2="73.66" y2="121.92" width="0.1524" layer="91"/>
+<junction x="73.66" y="124.46"/>
+<pinref part="C3" gate="G$1" pin="1"/>
+<pinref part="U$1" gate="G$1" pin="P0.01/XTAL2"/>
+<wire x1="48.26" y1="124.46" x2="73.66" y2="124.46" width="0.1524" layer="91"/>
+<wire x1="48.26" y1="124.46" x2="48.26" y2="73.66" width="0.1524" layer="91"/>
+</segment>
+</net>

Commit message: Adjustments
Connections:
- removed net D3: MS1.GPIOA3
- removed net D6: MS1.GPIOA1, U$1.P0.26
- new net P1.06: MS1.NC, U$1.P1.06
- net D2: now also MS1.GPIOA4
- net D4: now also MS1.GPIOA2, U$1.P0.06; no longer MS1.NC, U$1.P1.06
- net D5: now also MS1.GPIOA1, U$1.P0.26; no longer MS1.GPIOA2, U$1.P0.06
Other:
- note added: "We'll use the internal crystal connected to XC2, XC1"
- note added: "XTAL"
Changed lines of the file:
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@@
 <text x="195.58" y="17.78" size="1.778" layer="94">RED LED</text>
 <text x="215.9" y="17.78" size="1.778" layer="94">RESET</text>
+<text x="63.5" y="96.52" size="1.778" layer="94">XTAL</text>
+<text x="71.12" y="91.44" size="1.27" layer="97" align="center">We'll use the internal
+crystal connected to XC2, XC1</text>
 <text x="109.22" y="91.44" size="1.778" layer="94">MICRO USB</text>
 <text x="187.96" y="-40.64" size="1.778" layer="94">SPI Flash</text>
@@
 </segment>
 </net>
-<net name="D4" class="0">
+<net name="P1.06" class="0">
 <segment>
 <pinref part="MS1" gate="G$1" pin="NC"/>
@@
 <label x="-17.78" y="-43.18" size="1.778" layer="95"/>
 </segment>
-</net>
-<net name="D3" class="0">
-<segment>
-<pinref part="MS1" gate="G$1" pin="GPIOA3"/>
-<wire x1="-124.46" y1="-15.24" x2="-132.08" y2="-15.24" width="0.1524" layer="91"/>
-<label x="-129.54" y="-15.24" size="1.778" layer="95"/>
-</segment>
-</net>
-<net name="D5" class="0">
+<segment>
+<pinref part="MS1" gate="G$1" pin="GPIOA4"/>
+<wire x1="-124.46" y1="-17.78" x2="-132.08" y2="-17.78" width="0.1524" layer="91"/>
+<label x="-129.54" y="-17.78" size="1.778" layer="95"/>
+</segment>
+</net>
+<net name="D4" class="0">
 <segment>
 <pinref part="U$1" gate="G$1" pin="P0.06"/>
@@
 </segment>
 </net>
-<net name="D6" class="0">
+<net name="D5" class="0">
 <segment>
 <pinref part="U$1" gate="G$1" pin="P0.26"/>
